File: schematics/backplanev5/backplanev5.kicad_sch (KiCad schematic)
At the start: 0 parts

Commit message: Initial commit
Other:
- added sheet backplane (backplane.kicad_sch)
Changed lines of the file:
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@@
 	(generator_version "9.0")
 	(paper "A4")
+	(sheet
+		(at 25.4 38.1)
+		(size 76.2 16.51)
+		(exclude_from_sim no)
+		(in_bom yes)
+		(on_board yes)
+		(dnp no)
+		(fields_autoplaced yes)
+		(stroke
+			(width 0.1524)
+			(type solid)
+		)
+		(fill
+			(color 0 0 0 0.0000)
+		)
+		(property "Sheetname" "backplane"
+			(at 25.4 37.3884 0)
+			(effects
+				(font
+					(size 1.27 1.27)
+				)
+				(justify left bottom)
+			)
+		)
+		(property "Sheetfile" "backplane.kicad_sch"
+			(at 25.4 55.1946 0)
+			(effects
+				(font
+					(size 1.27 1.27)
+				)
+				(justify left top)
+			)
+		)
+		(instances
+			(project "backplanev5"
+				(path "/c4851f5c-edd8-4340-8a53-6aaa01d97892"
+					(page "2")
+				)
+			)
+		)
+	)
 	(sheet_instances
 		(path "/"
